File: 49er.sch (EAGLE design)
At the start: 47 parts, among them IC1 SA612AN, IC2 LM386N-1, IC3 78L05Z, Q1 2N5484, Q2 2N3904, Q3 2N3866, X1 7.040 MHz

Commit message: GND bug fix
Connections:
- removed net N$6: C2.A, C20.2, L1.2
- net GND: now also C2.A, C20.2, L1.2
Changed lines of the file:
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@@
 <part name="SUPPLY21" library="supply2" deviceset="GND" device=""/>
 <part name="JP3" library="pinhead" deviceset="PINHD-1X2" device="" value="KEY"/>
+<part name="SUPPLY22" library="supply2" deviceset="GND" device=""/>
 </parts>
 <sheets>
@@
 <instance part="SUPPLY21" gate="GND" x="144.78" y="127"/>
 <instance part="JP3" gate="G$1" x="91.44" y="12.7"/>
+<instance part="SUPPLY22" gate="GND" x="-5.08" y="93.98"/>
 </instances>
 <busses>
@@
 <pinref part="SUPPLY14" gate="GND" pin="GND"/>
 <wire x1="81.28" y1="12.7" x2="88.9" y2="12.7" width="0.1524" layer="91"/>
+</segment>
+<segment>
+<pinref part="L1" gate="G$1" pin="2"/>
+<junction x="2.54" y="96.52"/>
+<pinref part="C20" gate="G$1" pin="2"/>
+<wire x1="-15.24" y1="104.14" x2="-15.24" y2="96.52" width="0.1524" layer="91"/>
+<wire x1="-15.24" y1="96.52" x2="-5.08" y2="96.52" width="0.1524" layer="91"/>
+<pinref part="C2" gate="G$1" pin="A"/>
+<wire x1="-5.08" y1="96.52" x2="2.54" y2="96.52" width="0.1524" layer="91"/>
+<wire x1="-5.08" y1="104.14" x2="-5.08" y2="96.52" width="0.1524" layer="91"/>
+<junction x="-15.24" y="96.52"/>
+<junction x="-5.08" y="96.52"/>
+<pinref part="SUPPLY22" gate="GND" pin="GND"/>
 </segment>
 </net>
@@
 </segment>
 </net>
-<net name="N$6" class="0">
-<segment>
-<pinref part="L1" gate="G$1" pin="2"/>
-<junction x="2.54" y="96.52"/>
-<pinref part="C20" gate="G$1" pin="2"/>
-<wire x1="-15.24" y1="104.14" x2="-15.24" y2="96.52" width="0.1524" layer="91"/>
-<wire x1="-15.24" y1="96.52" x2="-5.08" y2="96.52" width="0.1524" layer="91"/>
-<pinref part="C2" gate="G$1" pin="A"/>
-<wire x1="-5.08" y1="96.52" x2="2.54" y2="96.52" width="0.1524" layer="91"/>
-<wire x1="-5.08" y1="104.14" x2="-5.08" y2="96.52" width="0.1524" layer="91"/>
-<junction x="-15.24" y="96.52"/>
-<junction x="-5.08" y="96.52"/>
-</segment>
-</net>
