File: 49er.brd (EAGLE design)
At the start: 88.6 x 53.3 mm, 47 parts, among them IC1 SA612AN, IC2 LM386N-1, IC3 78L05Z, Q1 2N5484, Q2 2N3904, Q3 2N3866, X1 7.040 MHz

Commit message: cambios menores
Parts:
- moved L6 47.4 mm to (34.3, 43.2), turned to 180 degrees
- moved C6 10.2 mm to (43.2, 41.9), turned to 90 degrees
- moved C7 6.48 mm to (12.7, 39.4)
- moved C1 6.35 mm to (6.35, 39.4)
- moved C2 4.58 mm to (6.35, 30.5)
- moved C20 4.02 mm to (14.0, 30.5)
- moved L2 3.81 mm to (76.2, 15.2)
- moved X1 3.59 mm to (34.3, 39.4)
- moved L1 2.54 mm to (10.2, 35.6)
- moved C8 1.27 mm to (33.0, 10.2)
Routing:
- net N$8: track 40.6 -> 7.14 mm
- net N$11: track 27.6 -> 4.41 mm
- net N$6: track 19.8 -> 13.1 mm
- net N$2: track 15.0 -> 8.67 mm
- net N$7: track 25.5 -> 27.3 mm
- net N$9: track 15.1 -> 13.4 mm
- net N$10: track 40.0 -> 38.4 mm
Other:
- board text added: "NorCal QRP 49er by N6KR PCB by LU4EXT"

Commit message: GND bug fix
Connections:
- removed net N$6: C2.-, C20.2, L1.2
- net GND: now also C2.-, C20.2, L1.2
Routing:
- net N$6: track 13.1 -> 0.00 mm
Changed lines of the file:
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@@
 <contactref element="JP2" pad="2"/>
 <contactref element="JP3" pad="2"/>
+<contactref element="L1" pad="2"/>
+<contactref element="C20" pad="2"/>
+<contactref element="C2" pad="-"/>
 </signal>
 <signal name="N$2">
@@
 <wire x1="5.08" y1="30.48" x2="4.475" y2="30.48" width="0.4064" layer="16"/>
 </signal>
-<signal name="N$6">
-<contactref element="L1" pad="2"/>
-<contactref element="C20" pad="2"/>
-<contactref element="C2" pad="-"/>
-<wire x1="15.24" y1="35.56" x2="15.24" y2="30.48" width="0.4064" layer="16"/>
-<wire x1="10.16" y1="30.48" x2="8.225" y2="30.48" width="0.4064" layer="16"/>
-<wire x1="11.43" y1="29.21" x2="10.16" y2="30.48" width="0.4064" layer="16"/>
-<wire x1="13.97" y1="29.21" x2="11.43" y2="29.21" width="0.4064" layer="16"/>
-<wire x1="15.24" y1="30.48" x2="13.97" y2="29.21" width="0.4064" layer="16"/>
-</signal>
 <signal name="N$7">

Commit message: GND bug fix
Routing:
- net GND: track 0.00 -> 11.4 mm
Changed lines of the file:
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@@
 <contactref element="C20" pad="2"/>
 <contactref element="C2" pad="-"/>
+<wire x1="8.89" y1="30.48" x2="8.89" y2="27.94" width="0.4064" layer="16"/>
+<wire x1="8.89" y1="27.94" x2="15.24" y2="27.94" width="0.4064" layer="16"/>
+<wire x1="15.24" y1="27.94" x2="15.24" y2="30.48" width="0.4064" layer="16"/>
 </signal>
 <signal name="N$2">
